Commit message: Rename wrist macro. Delete duplicated materials. Add combined urdf

File: tiago_description/urdf/arm/arm.urdf.xacro (robot description, xacro)
@@ -228,5 +228,5 @@
     <!--        WRIST           -->
     <!--************************-->
-    <xacro:wrist name="arm" parent="${name}_4_link" reflect="1"/>
+    <xacro:tiagowrist name="arm" parent="${name}_4_link" reflect="1"/>
     <!--***********************-->
     <!--        TOOL           -->

File: tiago_description/urdf/arm/wrist.urdf.xacro (robot description, xacro)
@@ -21,5 +21,5 @@
   <xacro:property name="wrist_3_max_effort"   value="6.6" />
   <xacro:property name="wrist_eps"          value="0.02" />
-  <xacro:macro name="wrist" params="name parent reflect">
+  <xacro:macro name="tiagowrist" params="name parent reflect">
     <!--************************-->
     <!--        WRIST           -->

File: tiago_description/urdf/materials.urdf.xacro (robot description, xacro)
@@ -8,25 +8,7 @@
 -->
 <robot>
-  <material name="Blue">
-    <color rgba="0.0 0.0 0.8 1.0"/>
-  </material>
-  <material name="Green">
-    <color rgba="0.0 0.8 0.0 1.0"/>
-  </material>
-  <material name="Grey">
-    <color rgba="0.7 0.7 0.7 1.0"/>
-  </material>
-  <material name="LightGrey">
-    <color rgba="0.9 0.9 0.9 1.0"/>
-  </material>
  <material name="DarkGrey">
    <color rgba="0.1 0.1 0.1 1.0"/>
  </material>
-  <material name="Red">
-    <color rgba="0.8 0.0 0.0 1.0"/>
-  </material>
-  <material name="White">
-    <color rgba="1.0 1.0 1.0 1.0"/>
-  </material>
   <material name="Yellow">
     <color rgba="0.96 0.88 0.14 1.0"/>
